File: Main/Main.kicad_sch (KiCad schematic)
At the start: 78 parts, among them J1 Conn_02x16_Odd_Even, J2 TYPE-C 6P, J3 Conn_01x02, Q3 S9013 J3(RANGE:200-350), SW2 SS-12D11G3R, U1 BQ24074RGT, U2 DRV8833PW, U3 HUSB237-AA001-DN06R, U4 RT9742GGJ5, U5 RT9742GGJ5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

Commit message: Using a new Motor Driver bc old one no stock
Parts:
- removed U2, U8: DRV8833PW, Package_SO:TSSOP-16_4.4x5mm_P0.65mm, symbol Driver_Motor:DRV8833PW
- added U10, U11: DRV8833PWP, Package_SO:HTSSOP-16-1EP_4.4x5mm_P0.65mm_EP3.4x5mm_Mask2.46x2.31mm_ThermalVias, symbol Driver_Motor:DRV8833PWP
- U6: footprint Package_TO_SOT_SMD:SOT-23-8 -> Package_TO_SOT_SMD:SOT-23-8_Handsoldering
Connections:
- net Battery: now also U10.12 (VM), U11.12 (VM)
- net GND: now also U10.13 (GND), U10.17 (GND), U11.13 (GND), U11.17 (GND)
- net MOTOR1_A_OUT: now also U11.2 (AOUT1)
- net MOTOR1_B_OUT: now also U11.4 (AOUT2)
- net MOTOR1_CTRL1: now also U11.16 (AIN1)
- net MOTOR1_CTRL2: now also U11.15 (AIN2)
- net MOTOR2_CTRL1: now also U11.9 (BIN1)
- net MOTOR2_CTRL2: now also U11.10 (BIN2)
- net MOTOR3_A_OUT: now also U10.2 (AOUT1)
- net MOTOR3_B_OUT: now also U10.4 (AOUT2)
- net MOTOR3_CTRL1: now also U10.16 (AIN1)
- net MOTOR3_CTRL2: now also U10.15 (AIN2)
- net MOTOR4_CTRL1: now also U10.9 (BIN1)
- net MOTOR4_CTRL2: now also U10.10 (BIN2)
- net Motor2_A_OUT: now also U11.7 (BOUT1)
- net Motor2_B_OUT: now also U11.5 (BOUT2)
- net Motor4_A_OUT: now also U10.7 (BOUT1)
- net Motor4_B_OUT: now also U10.5 (BOUT2)
- net at C5.2: now also U10.14 (VINT)
- net at R19.2: now also U10.1 (~{SLEEP})
- net at R3.2, TP1.1: now also U11.3 (AISEN), U11.6 (BISEN)
- net at R17.2, TP4.1: now also U10.3 (AISEN), U10.6 (BISEN)
- net at C6.2: now also U10.11 (VCP)
- net at R4.2: now also U11.1 (~{SLEEP})
- net at C3.2: now also U11.11 (VCP)
- net at C2.2: now also U11.14 (VINT)
Changed lines of the file:
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@@
 	)
 	(symbol
-		(lib_id "Driver_Motor:DRV8833PW")
-		(at 233.68 162.56 0)
-		(unit 1)
-		(exclude_from_sim no)
-		(in_bom yes)
-		(on_board yes)
-		(dnp no)
-		(fields_autoplaced yes)
-		(property "Reference" "U8"
-			(at 235.8233 177.8 0)
-			(effects
-				(font
-					(size 1.27 1.27)
-				)
-				(justify left)
-			)
-		)
-		(property "Value" "DRV8833PW"
-			(at 235.8233 180.34 0)
-			(effects
-				(font
-					(size 1.27 1.27)
-				)
-				(justify left)
-			)
-		)
-		(property "Footprint" "Package_SO:TSSOP-16_4.4x5mm_P0.65mm"
-			(at 238.76 180.34 0)
-			(effects
-				(font
-					(size 1.27 1.27)
-				)
-				(justify left)
-				(hide yes)
-			)
-		)
-		(property "Datasheet" "https://jlcpcb.com/api/file/downloadByFileSystemAccessId/8588881461298802689"
-			(at 238.76 182.88 0)
-			(effects
-				(font
-					(size 1.27 1.27)
-				)
-				(justify left)
-				(hide yes)
-			)
-		)
-		(property "Description" "Dual H-Bridge Motor Driver, TSSOP-16"
-			(at 233.68 162.56 0)
-			(effects
-				(font
-					(size 1.27 1.27)
-				)
-				(hide yes)
-			)
-		)
-		(property "LCSC" " C50506"
-			(at 233.68 162.56 0)
-			(effects
-				(font
-					(size 1.27 1.27)
-				)
-				(hide yes)
-			)
-		)
-		(pin "3"
-		)
-		(pin "11"
-		)
-		(pin "8"
-		)
-		(pin "1"
-		)
-		(pin "6"
-		)
-		(pin "16"
-		)
-		(pin "15"
-		)
-		(pin "9"
-		)
-		(pin "10"
-		)
-		(pin "13"
-		)
-		(pin "14"
-		)
-		(pin "12"
-		)
-		(pin "4"
-		)
-		(pin "7"
-		)
-		(pin "5"
-		)
-		(pin "2"
-		)
-		(instances
-			(project "Main"
-				(path "/0f55449c-8e79-4f10-a328-a1bcb934c334"
-					(reference "U8")
-					(unit 1)
-				)
-			)
-		)
-	)
-	(symbol
 		(lib_id "power:GND")
 		(at 163.83 104.14 270)
@@
 	)
 	(symbol
-		(lib_id "Driver_Motor:DRV8833PW")
-		(at 158.75 162.56 0)
-		(unit 1)
-		(exclude_from_sim no)
-		(in_bom yes)
-		(on_board yes)
-		(dnp no)
-		(fields_autoplaced yes)
-		(property "Reference" "U2"
-			(at 160.8933 177.8 0)
-			(effects
-				(font
-					(size 1.27 1.27)
-				)
-				(justify left)
-			)
-		)
-		(property "Value" "DRV8833PW"
-			(at 160.8933 180.34 0)
-			(effects
-				(font
-					(size 1.27 1.27)
-				)
-				(justify left)
-			)
-		)
-		(property "Footprint" "Package_SO:TSSOP-16_4.4x5mm_P0.65mm"
-			(at 163.83 180.34 0)
-			(effects
-				(font
-					(size 1.27 1.27)
-				)
-				(justify left)
-				(hide yes)
-			)
-		)
-		(property "Datasheet" "https://jlcpcb.com/api/file/downloadByFileSystemAccessId/8588881461298802689"
-			(at 163.83 182.88 0)
-			(effects
-				(font
-					(size 1.27 1.27)
-				)
-				(justify left)
-				(hide yes)
-			)
-		)
-		(property "Description" "Dual H-Bridge Motor Driver, TSSOP-16"
-			(at 158.75 162.56 0)
-			(effects
-				(font
-					(size 1.27 1.27)
-				)
-				(hide yes)
-			)
-		)
-		(property "LCSC" " C50506"
-			(at 158.75 162.56 0)
-			(effects
-				(font
-					(size 1.27 1.27)
-				)
-				(hide yes)
-			)
-		)
-		(pin "3"
-		)
-		(pin "11"
-		)
-		(pin "8"
-		)
-		(pin "1"
-		)
-		(pin "6"
-		)
-		(pin "16"
-		)
-		(pin "15"
-		)
-		(pin "9"
-		)
-		(pin "10"
-		)
-		(pin "13"
-		)
-		(pin "14"
-		)
-		(pin "12"
-		)
-		(pin "4"
-		)
-		(pin "7"
-		)
-		(pin "5"
-		)
-		(pin "2"
-		)
-		(instances
-			(project "Main"
-				(path "/0f55449c-8e79-4f10-a328-a1bcb934c334"
-					(reference "U2")
-					(unit 1)
-				)
-			)
-		)
-	)
-	(symbol
 		(lib_id "Device:R_Small_US")
 		(at 213.36 90.17 90)
@@
 	)
 	(symbol
+		(lib_id "Driver_Motor:DRV8833PWP")
+		(at 233.68 162.56 0)
+		(unit 1)
+		(exclude_from_sim no)
+		(in_bom yes)
+		(on_board yes)
+		(dnp no)
+		(fields_autoplaced yes)
+		(property "Reference" "U10"
+			(at 235.8233 177.8 0)
+			(effects
+				(font
+					(size 1.27 1.27)
+				)
+				(justify left)
+			)
+		)
+		(property "Value" "DRV8833PWP"
+			(at 235.8233 180.34 0)
+			(effects
+				(font
+					(size 1.27 1.27)
+				)
+				(justify left)
+			)
+		)
+		(property "Footprint" "Package_SO:HTSSOP-16-1EP_4.4x5mm_P0.65mm_EP3.4x5mm_Mask2.46x2.31mm_ThermalVias"
+			(at 238.76 177.8 0)
+			(effects
+				(font
+					(size 1.27 1.27)
+				)
+				(justify left)
+				(hide yes)
+			)
+		)
+		(property "Datasheet" "http://www.ti.com/lit/ds/symlink/drv8833.pdf"
+			(at 238.76 180.34 0)
+			(effects
+				(font
+					(size 1.27 1.27)
+				)
+				(justify left)
+				(hide yes)
+			)
+		)
+		(property "Description" "Dual H-Bridge Motor Driver, HTSSOP-16"
+			(at 233.68 162.56 0)
+			(effects
+				(font
+					(size 1.27 1.27)
+				)
+				(hide yes)
+			)
+		)
+		(property "LCSC" "C1556089"
+			(at 233.68 162.56 0)
+			(effects
+				(font
+					(size 1.27 1.27)
+				)
+				(hide yes)
+			)
+		)
+		(pin "3"
+		)
+		(pin "12"
+		)
+		(pin "2"
+		)
+		(pin "15"
+		)
+		(pin "4"
+		)
+		(pin "1"
+		)
+		(pin "8"
+		)
+		(pin "6"
+		)
+		(pin "11"
+		)
+		(pin "10"
+		)
+		(pin "17"
+		)
+		(pin "14"
+		)
+		(pin "16"
+		)
+		(pin "9"
+		)
+		(pin "13"
+		)
+		(pin "7"
+		)
+		(pin "5"
+		)
+		(instances
+			(project ""
+				(path "/0f55449c-8e79-4f10-a328-a1bcb934c334"
+					(reference "U10")
+					(unit 1)
+				)
+			)
+		)
+	)
+	(symbol
 		(lib_id "Device:C_Small")
 		(at 167.64 240.03 90)
@@
 	)
 	(symbol
+		(lib_id "Driver_Motor:DRV8833PWP")
+		(at 158.75 162.56 0)
+		(unit 1)
+		(exclude_from_sim no)
+		(in_bom yes)
+		(on_board yes)
+		(dnp no)
+		(fields_autoplaced yes)
+		(property "Reference" "U11"
+			(at 160.8933 177.8 0)
+			(effects
+				(font
+					(size 1.27 1.27)
+				)
+				(justify left)
+			)
+		)
+		(property "Value" "DRV8833PWP"
+			(at 160.8933 180.34 0)
+			(effects
+				(font
+					(size 1.27 1.27)
+				)
+				(justify left)
+			)
+		)
+		(property "Footprint" "Package_SO:HTSSOP-16-1EP_4.4x5mm_P0.65mm_EP3.4x5mm_Mask2.46x2.31mm_ThermalVias"
+			(at 163.83 177.8 0)
+			(effects
+				(font
+					(size 1.27 1.27)
+				)
+				(justify left)
+				(hide yes)
+			)
+		)
+		(property "Datasheet" "http://www.ti.com/lit/ds/symlink/drv8833.pdf"
+			(at 163.83 180.34 0)
+			(effects
+				(font
+					(size 1.27 1.27)
+				)
+				(justify left)
+				(hide yes)
+			)
+		)
+		(property "Description" "Dual H-Bridge Motor Driver, HTSSOP-16"
+			(at 158.75 162.56 0)
+			(effects
+				(font
+					(size 1.27 1.27)
+				)
+				(hide yes)
+			)
+		)
+		(property "LCSC" "C1556089"
+			(at 158.75 162.56 0)
+			(effects
+				(font
+					(size 1.27 1.27)
+				)
+				(hide yes)
+			)
+		)
+		(pin "3"
+		)
+		(pin "12"
+		)
+		(pin "2"
+		)
+		(pin "15"
+		)
+		(pin "4"
+		)
+		(pin "1"
+		)
+		(pin "8"
+		)
+		(pin "6"
+		)
+		(pin "11"
+		)
+		(pin "10"
+		)
+		(pin "17"
+		)
+		(pin "14"
+		)
+		(pin "16"
+		)
+		(pin "9"
+		)
+		(pin "13"
+		)
+		(pin "7"
+		)
+		(pin "5"
+		)
+		(instances
+			(project "Main"
+				(path "/0f55449c-8e79-4f10-a328-a1bcb934c334"
+					(reference "U11")
+					(unit 1)
+				)
+			)
+		)
+	)
+	(symbol
 		(lib_id "Device:R_Small_US")
 		(at 196.85 107.95 0)
@@
 			)
 		)
-		(property "Footprint" "Package_TO_SOT_SMD:SOT-23-8"
+		(property "Footprint" "Package_TO_SOT_SMD:SOT-23-8_Handsoldering"
 			(at 176.53 234.95 0)
 			(effects

Commit message: NO ERRORS
Parts:
- U10, U11: footprint Package_SO:HTSSOP-16-1EP_4.4x5mm_P0.65mm_EP3.4x5mm_Mask2.46x2.31mm_ThermalVias -> Package_SO:HTSSOP-16-1EP_4.4x5mm_P0.65mm_EP3.4x5mm_Mask2.46x2.31mm
Changed lines of the file:
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@@
 			)
 		)
-		(property "Footprint" "Package_SO:HTSSOP-16-1EP_4.4x5mm_P0.65mm_EP3.4x5mm_Mask2.46x2.31mm_ThermalVias"
+		(property "Footprint" "Package_SO:HTSSOP-16-1EP_4.4x5mm_P0.65mm_EP3.4x5mm_Mask2.46x2.31mm"
 			(at 238.76 177.8 0)
 			(effects
@@
 			)
 		)
-		(property "Footprint" "Package_SO:HTSSOP-16-1EP_4.4x5mm_P0.65mm_EP3.4x5mm_Mask2.46x2.31mm_ThermalVias"
+		(property "Footprint" "Package_SO:HTSSOP-16-1EP_4.4x5mm_P0.65mm_EP3.4x5mm_Mask2.46x2.31mm"
 			(at 163.83 177.8 0)
 			(effects
